Commit message: Fixed path to mesh

File: examples/urdf/coman.urdf (robot description, URDF)
Before this commit: robot coman, 65 links, 64 joints
Links:
- link DWL: geometry collision mesh filename=package://cartesian_interface/examples/mesh/coman/Torso1.STL scale=0.03937 0.03937 0.03937; visual mesh filename=package://cartesian_interface/examples/mesh/coman/Torso1.STL scale=0.03937 0.03937 0.03937
- link DWS: geometry collision mesh filename=package://cartesian_interface/examples/mesh/coman/Torso2.STL scale=0.03937 0.03937 0.03937; visual mesh filename=package://cartesian_interface/examples/mesh/coman/Torso2.STL scale=0.03937 0.03937 0.03937
- link DWYTorso: geometry collision mesh filename=package://cartesian_interface/examples/mesh/coman/Torso3.STL scale=0.03937 0.03937 0.03937; visual mesh filename=package://cartesian_interface/examples/mesh/coman/Torso3.STL scale=0.03937 0.03937 0.03937
- link LElb: geometry collision mesh filename=package://cartesian_interface/examples/mesh/coman/Elbow.STL scale=1.0 1.0 1.0; visual mesh filename=package://cartesian_interface/examples/mesh/coman/Elbow.STL scale=1.0 1.0 1.0
- link LFootmot: geometry collision mesh filename=package://cartesian_interface/examples/mesh/coman/Leg4.STL scale=0.03937 -0.03937 0.03937; visual mesh filename=package://cartesian_interface/examples/mesh/coman/Leg4.STL scale=0.03937 -0.03937 0.03937
- link LForearm: geometry collision mesh filename=package://cartesian_interface/examples/mesh/coman/Forearm0.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 scale=1.0 1.0 1.0; visual mesh filename=package://cartesian_interface/examples/mesh/coman/Forearm0.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 scale=0.1 0.1 0.1
- link LHipMot: geometry collision mesh filename=package://cartesian_interface/examples/mesh/coman/Leg0.STL scale=0.03937 -0.03937 0.03937; visual mesh filename=package://cartesian_interface/examples/mesh/coman/Leg0.STL scale=0.03937 -0.03937 0.03937
- link LLowLeg: geometry collision mesh filename=package://cartesian_interface/examples/mesh/coman/Leg3.STL scale=0.03937 -0.03937 0.03937; visual mesh filename=package://cartesian_interface/examples/mesh/coman/Leg3.STL scale=0.03937 -0.03937 0.03937
- link LShp: geometry collision mesh filename=package://cartesian_interface/examples/mesh/coman/Arm0.STL scale=0.03937 -0.03937 0.03937; visual mesh filename=package://cartesian_interface/examples/mesh/coman/Arm0.STL scale=0.03937 -0.03937 0.03937
- link LShr: geometry collision mesh filename=package://cartesian_interface/examples/mesh/coman/Arm1.STL scale=0.03937 -0.03937 0.03937; visual mesh filename=package://cartesian_interface/examples/mesh/coman/Arm1.STL scale=0.03937 -0.03937 0.03937
- link LShy: geometry collision mesh filename=package://cartesian_interface/examples/mesh/coman/Arm2.STL scale=0.03937 -0.03937 0.03937; visual mesh filename=package://cartesian_interface/examples/mesh/coman/Arm2.STL scale=0.03937 -0.03937 0.03937
- link LSoftHand: geometry collision mesh filename=package://cartesian_interface/examples/mesh/coman/SoftHandO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 scale=-1E-3 1E-3 1E-3; visual mesh filename=package://cartesian_interface/examples/mesh/coman/SoftHandO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 scale=-0.1 0.1 0.1
- link LThighLowLeg: geometry collision mesh filename=package://cartesian_interface/examples/mesh/coman/Leg2.STL scale=0.03937 -0.03937 0.03937; visual mesh filename=package://cartesian_interface/examples/mesh/coman/Leg2.STL scale=0.03937 -0.03937 0.03937
- link LThighUpLeg: geometry collision mesh filename=package://cartesian_interface/examples/mesh/coman/Leg1.STL scale=0.03937 -0.03937 0.03937; visual mesh filename=package://cartesian_interface/examples/mesh/coman/Leg1.STL scale=0.03937 -0.03937 0.03937
- link LWrMot2: geometry collision mesh filename=package://cartesian_interface/examples/mesh/coman/Forearm1.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 scale=0.001 0.001 0.001; visual mesh filename=package://cartesian_interface/examples/mesh/coman/Forearm1.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 scale=0.001 0.001 0.001
- link LWrMot3: geometry collision mesh filename=package://cartesian_interface/examples/mesh/coman/Forearm2.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 scale=0.001 0.001 0.001; visual mesh filename=package://cartesian_interface/examples/mesh/coman/Forearm2.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 scale=0.001 0.001 0.001
- link RElb: geometry collision mesh filename=package://cartesian_interface/examples/mesh/coman/Elbow.STL scale=1.0 1.0 1.0; visual mesh filename=package://cartesian_interface/examples/mesh/coman/Elbow.STL scale=1.0 1.0 1.0
- link RFootmot: geometry collision mesh filename=package://cartesian_interface/examples/mesh/coman/Leg4.STL scale=0.03937 0.03937 0.03937; visual mesh filename=package://cartesian_interface/examples/mesh/coman/Leg4.STL scale=0.03937 0.03937 0.03937
- link RForearm: geometry collision mesh filename=package://cartesian_interface/examples/mesh/coman/Forearm0.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 scale=1.0 1.0 1.0; visual mesh filename=package://cartesian_interface/examples/mesh/coman/Forearm0.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 scale=0.1 0.1 0.1
- link RHipMot: geometry collision mesh filename=package://cartesian_interface/examples/mesh/coman/Leg0.STL scale=0.03937 0.03937 0.03937; visual mesh filename=package://cartesian_interface/examples/mesh/coman/Leg0.STL scale=0.03937 0.03937 0.03937
- link RLowLeg: geometry collision mesh filename=package://cartesian_interface/examples/mesh/coman/Leg3.STL scale=0.03937 0.03937 0.03937; visual mesh filename=package://cartesian_interface/examples/mesh/coman/Leg3.STL scale=0.03937 0.03937 0.03937
- link RShp: geometry collision mesh filename=package://cartesian_interface/examples/mesh/coman/Arm0.STL scale=0.03937 0.03937 0.03937; visual mesh filename=package://cartesian_interface/examples/mesh/coman/Arm0.STL scale=0.03937 0.03937 0.03937
- link RShr: geometry collision mesh filename=package://cartesian_interface/examples/mesh/coman/Arm1.STL scale=0.03937 0.03937 0.03937; visual mesh filename=package://cartesian_interface/examples/mesh/coman/Arm1.STL scale=0.03937 0.03937 0.03937
- link RShy: geometry collision mesh filename=package://cartesian_interface/examples/mesh/coman/Arm2.STL scale=0.03937 0.03937 0.03937; visual mesh filename=package://cartesian_interface/examples/mesh/coman/Arm2.STL scale=0.03937 0.03937 0.03937
- link RSoftHand: geometry collision mesh filename=package://cartesian_interface/examples/mesh/coman/SoftHandO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 scale=1E-3 1E-3 1E-3; visual mesh filename=package://cartesian_interface/examples/mesh/coman/SoftHandO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 scale=0.1 0.1 0.1
- link RThighLowLeg: geometry collision mesh filename=package://cartesian_interface/examples/mesh/coman/Leg2.STL scale=0.03937 0.03937 0.03937; visual mesh filename=package://cartesian_interface/examples/mesh/coman/Leg2.STL scale=0.03937 0.03937 0.03937
- link RThighUpLeg: geometry collision mesh filename=package://cartesian_interface/examples/mesh/coman/Leg1.STL scale=0.03937 0.03937 0.03937; visual mesh filename=package://cartesian_interface/examples/mesh/coman/Leg1.STL scale=0.03937 0.03937 0.03937
- link RWrMot2: geometry collision mesh filename=package://cartesian_interface/examples/mesh/coman/Forearm1.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 scale=0.001 0.001 0.001; visual mesh filename=package://cartesian_interface/examples/mesh/coman/Forearm1.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 scale=0.001 0.001 0.001
- link RWrMot3: geometry collision mesh filename=package://cartesian_interface/examples/mesh/coman/Forearm2.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 scale=0.001 0.001 0.001; visual mesh filename=package://cartesian_interface/examples/mesh/coman/Forearm2.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 scale=0.001 0.001 0.001
- link Waist: geometry collision mesh filename=package://cartesian_interface/examples/mesh/coman/Waist.STL scale=0.03937 0.03937 0.03937; visual mesh filename=package://cartesian_interface/examples/mesh/coman/Waist.STL scale=0.03937 0.03937 0.03937

Commit message: Fixed meshes

File: examples/urdf/coman.urdf (robot description, URDF)
Before this commit: robot coman, 65 links, 64 joints
Links:
- link LForearm: geometry collision mesh filename=package://cartesian_interface/examples/mesh/coman/Forearm0.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 scale=1.0 1.0 1.0; visual mesh filename=package://cartesian_interface/examples/mesh/coman/Forearm0.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 scale=1.0 1.0 1.0
- link LSoftHand: geometry collision mesh filename=package://cartesian_interface/examples/mesh/coman/SoftHandO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 scale=-1E-3 1E-3 1E-3; visual mesh filename=package://cartesian_interface/examples/mesh/coman/SoftHandO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 scale=-1E-3 1E-3 1E-3
- link RForearm: geometry collision mesh filename=package://cartesian_interface/examples/mesh/coman/Forearm0.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 scale=1.0 1.0 1.0; visual mesh filename=package://cartesian_interface/examples/mesh/coman/Forearm0.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 scale=1.0 1.0 1.0
- link RSoftHand: geometry collision mesh filename=package://cartesian_interface/examples/mesh/coman/SoftHandO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 scale=1E-3 1E-3 1E-3; visual mesh filename=package://cartesian_interface/examples/mesh/coman/SoftHandO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 scale=1E-3 1E-3 1E-3

Commit message: increased weights of hands in coman by 1 kg

File: examples/urdf/coman.urdf (robot description, URDF)
Before this commit: robot coman, 65 links, 64 joints
Links:
- link LSoftHand: mass 0.3 -> 1.3
- link RSoftHand: mass 0.3 -> 1.3
